Commit message: Update MH180 inertial origins, and R and U link stls.

File: motoman_mh_support/urdf/mh180.xacro (robot description, xacro)
@@ -1,5 +1,12 @@
 <?xml version="1.0" ?>
 <robot name="motoman_mh180" xmlns:xacro="http://ros.org/wiki/xacro">
+  <xacro:include filename="$(find motoman_mh_support)/urdf/common.gazebo"/>
   <xacro:include filename="$(find motoman_mh_support)/urdf/mh180_macro.xacro"/>
+  <link name="world">
+  </link>
+  <joint name="world_joint" type="fixed">
+    <parent link="world" />
+    <child link="base_link" />
+  </joint>
   <xacro:motoman_mh180 prefix=""/>
 </robot>

File: motoman_mh_support/urdf/mh180_macro.xacro (robot description, xacro)
@@ -49,5 +49,5 @@
     </collision>
     <inertial>
-      <origin xyz="0.0971 0.0684 0.4991"/>
+      <origin xyz="0.0971 0.0684 0.1571"/>
       <mass value="265.3"/>
       <inertia ixx="9.922" iyy="17.39" izz="18.37" iyz="1.933" ixz="1.549" ixy="2.22"/>
@@ -67,5 +67,5 @@
     </collision>
     <inertial>
-      <origin xyz="0.3213 -0.0395 1.035"/>
+      <origin xyz="-0.0037 -0.0395 0.3847"/>
       <mass value="193.4"/>
       <inertia ixx="36.23" iyy="35.91" izz="3.082" iyz="-2.634" ixz="-0.1331" ixy="-0.0251"/>
@@ -85,5 +85,5 @@
     </collision>
     <inertial>
-      <origin xyz="0.5059 0.039 1.9577"/>
+      <origin xyz="0.1809 0.039 0.1577"/>
       <mass value="258.7"/>
       <inertia ixx="9.447" iyy="28.96" izz="25.15" iyz="-1.596" ixz="6.1" ixy="-1.233"/>
@@ -103,5 +103,5 @@
     </collision>
     <inertial>
-      <origin xyz="1.516 -0.06 2.1"/>
+      <origin xyz="0.1583 -0.06 0"/>
       <mass value="22.63"/>
       <inertia ixx="0.1083" iyy="0.1802" izz="0.1954" iyz="0.0001" ixz="-0.0001" ixy="-0.0481"/>
@@ -121,5 +121,5 @@
     </collision>
     <inertial>
-      <origin xyz="1.6501 -0.0089 2.1"/>
+      <origin xyz="0.1001 -0.0089 0"/>
       <mass value="19.98"/>
       <inertia ixx="0.1421" iyy="0.1845" izz="0.238" iyz="-0.0001" ixz="0" ixy="0.0185"/>
@@ -143,5 +143,5 @@
     </collision>
     <inertial>
-      <origin xyz="1.765 -0.0012 2.1"/>
+      <origin xyz="0.014 0 0"/>
       <mass value="1.703"/>
       <inertia ixx="0.0065" iyy="0.0035" izz="0.0035" iyz="0" ixz="0" ixy="0"/>
@@ -162,4 +162,5 @@
       velocity="${TO_RADIANS * 125}"/>
   </joint>
+  <!-- Note: Increased effort to account for gas shock between links S and L. -->
   <joint name="${prefix}joint_2" type="revolute">
     <origin xyz="0.325 0 0.308"/>
@@ -170,5 +171,5 @@
       lower="${l_lower_limit}"
       upper="${l_upper_limit}"
-      effort="${23.5 * 120}"
+      effort="${23.5 * 300}"
       velocity="${TO_RADIANS * 115}"/>
   </joint>
